File: atmega16m1-breakout.brd (EAGLE design)
At the start: 25.4 x 38.1 mm, 19 parts, among them U501 MCP2551, U503 ATMEL16/32/64M1-AI, X500 16 MHz

Commit message: Oh yeah. BOM. And BOM cleanup.
Parts:
- R501: value NP -> 120
Changed lines of the file:
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@@
 <attribute name="VALUE" x="22.352" y="16.764" size="1.27" layer="27" rot="R90"/>
 </element>
-<element name="R501" library="rcl_custom" package="0603-B-NOSILK" value="NP" x="18.288" y="30.988" smashed="yes" rot="R270">
+<element name="R501" library="rcl_custom" package="0603-B-NOSILK" value="120" x="18.288" y="30.988" smashed="yes" rot="R270">
 <attribute name="NAME" x="19.812" y="29.845" size="0.635" layer="25" font="vector" ratio="20" rot="R90"/>
 <attribute name="VALUE" x="16.383" y="31.623" size="1.27" layer="27" rot="R270"/>
