File: atmega16m1-breakout.sch (EAGLE design)
At the start: 19 parts, among them U501 MCP2551, U503 ATMEL16/32/64M1-AI, X500 16 MHz

Commit message: Oh yeah. BOM. And BOM cleanup.
Parts:
- R501: value NP -> 120
Changed lines of the file:
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@@
 <part name="C502" library="rcl_custom" deviceset="C-EU" device="0603-B-NOSILK" value="100n"/>
 <part name="R502" library="rcl_custom" deviceset="R-US_" device="0603-B-NOSILK" value="10"/>
-<part name="R501" library="rcl_custom" deviceset="R-US_" device="0603-B-NOSILK" value="NP"/>
+<part name="R501" library="rcl_custom" deviceset="R-US_" device="0603-B-NOSILK" value="120"/>
 <part name="C500" library="rcl_custom" deviceset="C-EU" device="0603-B-NOSILK" value="1n"/>
 <part name="C501" library="rcl_custom" deviceset="C-EU" device="0805-B-NOSILK" value="10u"/>
